File: schematics/Arduino Nano Controller v1.0.kicad_pcb (KiCad board)
At the start: 2 copper layers, 48.3 x 57.2 mm, 5 parts, among them J1 H4, U1 H3

Commit message: Slight Refactoring
Parts:
- removed J1: H4, Connector_PinHeader_2.54mm:PinHeader_1x02_P2.54mm_Vertical
- added REF**: PinHeader_1x03_P2.54mm_Vertical, Connector_PinHeader_2.54mm:PinHeader_1x03_P2.54mm_Vertical, F.Cu at (170.2, 45.7)
- added S1: S1, Connector_PinHeader_2.54mm:PinHeader_1x03_P2.54mm_Vertical, F.Cu at (151.1, 68.6)
- moved 5V 5.08 mm to (135.9, 76.2)
Routing:
- net (no net): track 880.9 -> 656.7 mm
Other:
- board text added: "MODCOMP Controller v1.0 2020 Josh Heaton"
- board text removed: "MODCOMP 7830 Controller v1.1 2020 Josh Heaton"
